File: RPiPico_SimpleBoard.kicad_pcb (KiCad board)
At the start: 2 copper layers, 82.2 x 54 mm, 13 parts, among them J1 Conn_01x20, J2 Conn_01x20, J3 Conn_01x20, J4 Conn_01x20, J5 Debug, J6 Conn_01x04, SW1 SW_Push, U1 RaspberryPi_Pico

Commit message: Fix outline not to conflict with USB cables.
Parts:
- H1, H2, H3, H4: footprint MountingHole:MountingHole_3.2mm_M3_DIN965_Pad -> MountingHole:MountingHole_3.2mm_M3
Routing:
- net GND: track 56.1 -> 6.35 mm, vias 103 -> 98
Other:
- outline, holes or cut-outs redrawn
- board text added: "RPiPico Debug Board Rev.B 2023-02-19 @ciniml"
- board text removed: "RPiPico Probe Board Rev.A 2023-02-07 @ciniml"

Commit message: fix some silk prints
(GP5) U0RX -> U1RX
(GP26) I1SCL -> I1SDA
(GP21) GP20 -> GP21
Other:
- board text added: "I0SCL GP21"
- board text added: "I1SDA ADC0,GP26"
- board text added: "U1RX,I0SCL S0CSn,GP5"
- board text removed: "I0SCL GP20"
- board text removed: "I1SCL ADC0,GP26"
- board text removed: "U0RX,I0SCL S0CSn,GP5"
Changed lines of the file:
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@@
     (effects (font (size 0.8 0.8) (thickness 0.15)) (justify left))
   )
-  (gr_text "I0SCL\nGP20" (at 30.48 3.81 90) (layer "F.SilkS")
+  (gr_text "I0SCL\nGP21" (at 30.48 3.81 90) (layer "F.SilkS")
     (effects (font (size 0.8 0.8) (thickness 0.15)) (justify left))
   )
@@
     (effects (font (size 0.8 0.8) (thickness 0.15)) (justify left))
   )
-  (gr_text "U0RX,I0SCL\nS0CSn,GP5" (at 12.7 39.37 90) (layer "F.SilkS")
+  (gr_text "U1RX,I0SCL\nS0CSn,GP5" (at 12.7 39.37 90) (layer "F.SilkS")
     (effects (font (size 0.8 0.8) (thickness 0.15)) (justify right))
   )
@@
     (effects (font (size 0.8 0.8) (thickness 0.15)) (justify left))
   )
-  (gr_text "I1SCL\nADC0,GP26" (at 20.32 3.81 90) (layer "F.SilkS")
+  (gr_text "I1SDA\nADC0,GP26" (at 20.32 3.81 90) (layer "F.SilkS")
     (effects (font (size 0.8 0.8) (thickness 0.15)) (justify left))
   )

Commit message: Rev.C
Other:
- board text added: "RPiPico Debug Board Rev.C 2023-05-10 @ciniml"
- board text removed: "RPiPico Debug Board Rev.B 2023-02-19 @ciniml"
Changed lines of the file:
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@@
     (effects (font (size 0.8 0.8) (thickness 0.15)) (justify right))
   )
-  (gr_text "RPiPico\nDebug Board\nRev.B\n2023-02-19\n@ciniml" (at 48.895 35.56) (layer "F.SilkS")
+  (gr_text "RPiPico\nDebug Board\nRev.C\n2023-05-10\n@ciniml" (at 48.895 35.56) (layer "F.SilkS")
     (effects (font (size 1 1) (thickness 0.15)) (justify left))
   )
