File: RPiPico_SimpleBoard.kicad_sch (KiCad schematic)
At the start: 13 parts, among them J1 Conn_01x20, J2 Conn_01x20, J3 Conn_01x20, J4 Conn_01x20, J5 Debug, J6 Conn_01x04, SW1 SW_Push, U1 RaspberryPi_Pico

Commit message: Fix outline not to conflict with USB cables.
Parts:
- H1, H2, H3, H4: footprint MountingHole:MountingHole_3.2mm_M3_DIN965_Pad -> MountingHole:MountingHole_3.2mm_M3
Other:
- title: 1000BASE-T RGMII Ethernet Board -> RPi Pico Debug Board
